Commit message: Allow changing gpio_config.xacro

File: kuka_iontec_support/urdf/kr_iontec_ros2_control_macro.xacro (robot description, xacro)
@@ -1,5 +1,5 @@
 <?xml version="1.0" encoding="UTF-8"?>
 <robot xmlns:xacro="http://www.ros.org/wiki/xacro">
-  <xacro:macro name="kuka_iontec_ros2_control" params="name driver_version client_ip client_port mxa_client_port controller_ip prefix mode use_gpio roundtrip_time verify_robot_model **ext_axes_ros2_control_joints">
+  <xacro:macro name="kuka_iontec_ros2_control" params="name driver_version client_ip client_port mxa_client_port controller_ip prefix mode use_gpio roundtrip_time verify_robot_model gpio_config **ext_axes_ros2_control_joints">
     <!-- gazebo -->
     <xacro:if value="${mode == 'gazebo'}">
@@ -82,5 +82,5 @@
       </joint>
       <xacro:if value="${use_gpio}">
-        <xacro:include filename="$(find kuka_rsi_driver)/config/gpio_config.xacro"/>
+        <xacro:include filename="${gpio_config}"/>
         <xacro:gpio_config/>
       </xacro:if>
