Commit message: Update ros2control macro

File: kuka_iontec_support/urdf/kr_iontec_ros2_control_macro.xacro (robot description, xacro)
@@ -1,9 +1,9 @@
 <?xml version="1.0" encoding="UTF-8"?>
 <robot xmlns:xacro="http://www.ros.org/wiki/xacro">
-  <xacro:macro name="kuka_iontec_ros2_control" params="name driver_version client_ip client_port mxa_client_port controller_ip prefix mode use_gpio roundtrip_time verify_robot_model gpio_config **ext_axes_ros2_control_joints">
+  <xacro:macro name="kuka_iontec_ros2_control" params="name driver_version client_ip client_port mxa_client_port controller_ip prefix mode use_gpio roundtrip_time verify_robot_model rsi_xml_config_file gazebo_controller_config_path:=config/fake_hardware_config_6_axis.yaml gpio_config **ext_axes_ros2_control_joints">
     <!-- gazebo -->
     <xacro:if value="${mode == 'gazebo'}">
       <xacro:include filename="$(find kuka_gazebo)/gazebo/kuka_gazebo.xacro"/>
-      <xacro:kuka_gazebo controller_config_package="kuka_resources" controller_config_path="config/fake_hardware_config_6_axis.yaml"/>
+      <xacro:kuka_gazebo controller_config_package="kuka_resources" controller_config_path="${gazebo_controller_config_path}"/>
     </xacro:if>
     <!-- ros2 control -->
@@ -26,4 +26,5 @@
             <param name="name">${name}</param>
             <param name="verify_robot_model">${verify_robot_model}</param>
+            <param name="rsi_xml_config_file">${rsi_xml_config_file}</param>
           </xacro:if>
           <xacro:if value="${driver_version == 'mxa_rsi'}">
@@ -34,4 +35,5 @@
             <param name="mxa_client_port">${mxa_client_port}</param>
             <param name="verify_robot_model">${verify_robot_model}</param>
+            <param name="rsi_xml_config_file">${rsi_xml_config_file}</param>
           </xacro:if>
           <xacro:if value="${driver_version == 'rsi_only'}">
@@ -39,4 +41,5 @@
             <param name="client_ip">${client_ip}</param>
             <param name="client_port">${client_port}</param>
+            <param name="rsi_xml_config_file">${rsi_xml_config_file}</param>
           </xacro:if>
         </xacro:if>
@@ -48,61 +51,97 @@
       <joint name="${prefix}joint_1">
         <command_interface name="position"/>
-        <command_interface name="velocity"/>
-        <command_interface name="effort"/>
         <state_interface name="position">
           <param name="initial_value">0.0</param>
         </state_interface>
-        <state_interface name="velocity"/>
-        <state_interface name="effort"/>
+        <xacro:unless value="${mode == 'gazebo'}">
+          <command_interface name="velocity"/>
+          <command_interface name="effort"/>
+          <state_interface name="velocity">
+            <param name="initial_value">0.0</param>
+          </state_interface>
+          <state_interface name="effort">
+            <param name="initial_value">0.0</param>
+          </state_interface>
+        </xacro:unless>
       </joint>
       <joint name="${prefix}joint_2">
         <command_interface name="position"/>
-        <command_interface name="velocity"/>
-        <command_interface name="effort"/>
         <state_interface name="position">
           <param name="initial_value">-1.5708</param>
         </state_interface>
-        <state_interface name="velocity"/>
-        <state_interface name="effort"/>
+        <xacro:unless value="${mode == 'gazebo'}">
+          <command_interface name="velocity"/>
+          <command_interface name="effort"/>
+          <state_interface name="velocity">
+            <param name="initial_value">0.0</param>
+          </state_interface>
+          <state_interface name="effort">
+            <param name="initial_value">0.0</param>
+          </state_interface>
+        </xacro:unless>
       </joint>
       <joint name="${prefix}joint_3">
         <command_interface name="position"/>
-        <command_interface name="velocity"/>
-        <command_interface name="effort"/>
         <state_interface name="position">
           <param name="initial_value">1.5708</param>
         </state_interface>
-        <state_interface name="velocity"/>
-        <state_interface name="effort"/>
+        <xacro:unless value="${mode == 'gazebo'}">
+          <command_interface name="velocity"/>
+          <command_interface name="effort"/>
+          <state_interface name="velocity">
+            <param name="initial_value">0.0</param>
+          </state_interface>
+          <state_interface name="effort">
+            <param name="initial_value">0.0</param>
+          </state_interface>
+        </xacro:unless>
       </joint>
       <joint name="${prefix}joint_4">
         <command_interface name="position"/>
-        <command_interface name="velocity"/>
-        <command_interface name="effort"/>
         <state_interface name="position">
           <param name="initial_value">0.0</param>
         </state_interface>
-        <state_interface name="velocity"/>
-        <state_interface name="effort"/>
+        <xacro:unless value="${mode == 'gazebo'}">
+          <command_interface name="velocity"/>
+          <command_interface name="effort"/>
+          <state_interface name="velocity">
+            <param name="initial_value">0.0</param>
+          </state_interface>
+          <state_interface name="effort">
+            <param name="initial_value">0.0</param>
+          </state_interface>
+        </xacro:unless>
       </joint>
       <joint name="${prefix}joint_5">
         <command_interface name="position"/>
-        <command_interface name="velocity"/>
-        <command_interface name="effort"/>
         <state_interface name="position">
           <param name="initial_value">0.0</param>
         </state_interface>
-        <state_interface name="velocity"/>
-        <state_interface name="effort"/>
+        <xacro:unless value="${mode == 'gazebo'}">
+          <command_interface name="velocity"/>
+          <command_interface name="effort"/>
+          <state_interface name="velocity">
+            <param name="initial_value">0.0</param>
+          </state_interface>
+          <state_interface name="effort">
+            <param name="initial_value">0.0</param>
+          </state_interface>
+        </xacro:unless>
       </joint>
       <joint name="${prefix}joint_6">
         <command_interface name="position"/>
-        <command_interface name="velocity"/>
-        <command_interface name="effort"/>
         <state_interface name="position">
           <param name="initial_value">0.0</param>
         </state_interface>
-        <state_interface name="velocity"/>
-        <state_interface name="effort"/>
+        <xacro:unless value="${mode == 'gazebo'}">
+          <command_interface name="velocity"/>
+          <command_interface name="effort"/>
+          <state_interface name="velocity">
+            <param name="initial_value">0.0</param>
+          </state_interface>
+          <state_interface name="effort">
+            <param name="initial_value">0.0</param>
+          </state_interface>
+        </xacro:unless>
       </joint>
       <xacro:if value="${use_gpio}">

Commit message: Update ros2_control macros

File: kuka_iontec_support/urdf/kr_iontec_ros2_control_macro.xacro (robot description, xacro)
@@ -1,5 +1,5 @@
 <?xml version="1.0" encoding="UTF-8"?>
 <robot xmlns:xacro="http://www.ros.org/wiki/xacro">
-  <xacro:macro name="kuka_iontec_ros2_control" params="name driver_version client_ip client_port mxa_client_port controller_ip prefix mode use_gpio roundtrip_time verify_robot_model rsi_xml_config_file gazebo_controller_config_path:=config/fake_hardware_config_6_axis.yaml gpio_config **ext_axes_ros2_control_joints">
+  <xacro:macro name="kuka_iontec_ros2_control" params="name driver_version client_ip client_port mxa_client_port controller_ip prefix mode use_gpio roundtrip_time verify_robot_model rsi_xml_config_file is_async async_thread_priority async_affinity gazebo_controller_config_path:=config/fake_hardware_config_6_axis.yaml gpio_config:='' **ext_axes_ros2_control_joints">
     <!-- gazebo -->
     <xacro:if value="${mode == 'gazebo'}">
@@ -8,5 +8,8 @@
     </xacro:if>
     <!-- ros2 control -->
-    <ros2_control name="${name}" type="system">
+    <ros2_control name="${name}" type="system" is_async="${is_async}">
+      <properties>
+        <async affinity="${async_affinity}" scheduling_policy="detached" print_warnings="false" thread_priority="${async_thread_priority}"/>
+      </properties>
       <hardware>
         <param name="interface_prefix">${prefix}</param>
@@ -54,4 +57,14 @@
           <param name="initial_value">0.0</param>
         </state_interface>
+        <xacro:unless value="${mode == 'gazebo'}">
+          <command_interface name="velocity"/>
+          <command_interface name="effort"/>
+          <state_interface name="velocity">
+            <param name="initial_value">0.0</param>
+          </state_interface>
+          <state_interface name="effort">
+            <param name="initial_value">0.0</param>
+          </state_interface>
+        </xacro:unless>
       </joint>
       <joint name="${prefix}joint_2">
@@ -60,4 +73,14 @@
           <param name="initial_value">-1.5708</param>
         </state_interface>
+        <xacro:unless value="${mode == 'gazebo'}">
+          <command_interface name="velocity"/>
+          <command_interface name="effort"/>
+          <state_interface name="velocity">
+            <param name="initial_value">0.0</param>
+          </state_interface>
+          <state_interface name="effort">
+            <param name="initial_value">0.0</param>
+          </state_interface>
+        </xacro:unless>
       </joint>
       <joint name="${prefix}joint_3">
@@ -66,4 +89,14 @@
           <param name="initial_value">1.5708</param>
         </state_interface>
+        <xacro:unless value="${mode == 'gazebo'}">
+          <command_interface name="velocity"/>
+          <command_interface name="effort"/>
+          <state_interface name="velocity">
+            <param name="initial_value">0.0</param>
+          </state_interface>
+          <state_interface name="effort">
+            <param name="initial_value">0.0</param>
+          </state_interface>
+        </xacro:unless>
       </joint>
       <joint name="${prefix}joint_4">
@@ -72,4 +105,14 @@
           <param name="initial_value">0.0</param>
         </state_interface>
+        <xacro:unless value="${mode == 'gazebo'}">
+          <command_interface name="velocity"/>
+          <command_interface name="effort"/>
+          <state_interface name="velocity">
+            <param name="initial_value">0.0</param>
+          </state_interface>
+          <state_interface name="effort">
+            <param name="initial_value">0.0</param>
+          </state_interface>
+        </xacro:unless>
       </joint>
       <joint name="${prefix}joint_5">
@@ -78,4 +121,14 @@
           <param name="initial_value">0.0</param>
         </state_interface>
+        <xacro:unless value="${mode == 'gazebo'}">
+          <command_interface name="velocity"/>
+          <command_interface name="effort"/>
+          <state_interface name="velocity">
+            <param name="initial_value">0.0</param>
+          </state_interface>
+          <state_interface name="effort">
+            <param name="initial_value">0.0</param>
+          </state_interface>
+        </xacro:unless>
       </joint>
       <joint name="${prefix}joint_6">
@@ -84,4 +137,14 @@
           <param name="initial_value">0.0</param>
         </state_interface>
+        <xacro:unless value="${mode == 'gazebo'}">
+          <command_interface name="velocity"/>
+          <command_interface name="effort"/>
+          <state_interface name="velocity">
+            <param name="initial_value">0.0</param>
+          </state_interface>
+          <state_interface name="effort">
+            <param name="initial_value">0.0</param>
+          </state_interface>
+        </xacro:unless>
       </joint>
       <xacro:if value="${use_gpio}">

File: kuka_kl_support/urdf/kl_ros2_control_macro.xacro (robot description, xacro)
@@ -1,16 +1,22 @@
 <?xml version="1.0" encoding="UTF-8"?>
 <robot xmlns:xacro="http://www.ros.org/wiki/xacro">
-  <xacro:macro name="kuka_kl_ros2_control_joints" params="">
+  <xacro:macro name="kuka_kl_ros2_control_joints" params="mode">
     <joint name="rail_joint">
       <param name="type">prismatic</param>
       <param name="is_external">true</param>
       <command_interface name="position"/>
-      <!-- <command_interface name="velocity"/>
-      <command_interface name="effort"/> -->
       <state_interface name="position">
         <param name="initial_value">0.0</param>
       </state_interface>
-      <!-- <state_interface name="velocity"/>
-      <state_interface name="effort"/> -->
+      <xacro:unless value="${mode == 'gazebo'}">
+        <command_interface name="velocity"/>
+        <command_interface name="effort"/>
+        <state_interface name="velocity">
+          <param name="initial_value">0.0</param>
+        </state_interface>
+        <state_interface name="effort">
+          <param name="initial_value">0.0</param>
+        </state_interface>
+      </xacro:unless>
     </joint>
   </xacro:macro>
