Commit message: Add external axis support for k50_r2100

File: kuka_iontec_support/urdf/kr50_r2100.urdf.xacro (robot description, xacro)
@@ -11,4 +11,5 @@
   <xacro:arg name="client_ip" default="0.0.0.0"/>
   <xacro:arg name="client_port" default="59152"/>
+  <xacro:arg name="mxa_client_port" default="1337"/>
   <xacro:arg name="controller_ip" default="0.0.0.0"/>
   <xacro:arg name="verify_robot_model" default="true"/>
@@ -20,7 +21,17 @@
   <xacro:arg name="pitch" default="0"/>
   <xacro:arg name="yaw" default="0"/>
-  <xacro:kuka_iontec_ros2_control name="$(arg prefix)kr50_r2100" driver_version="$(arg driver_version)" client_ip="$(arg client_ip)" controller_ip="$(arg controller_ip)" client_port="$(arg client_port)" prefix="$(arg prefix)" mode="$(arg mode)" use_gpio="$(arg use_gpio)" roundtrip_time="$(arg roundtrip_time)" verify_robot_model="$(arg verify_robot_model)"/>
-  <xacro:kuka_kr50_r2100_robot prefix="$(arg prefix)" package_name="kuka_iontec_support">
+  <xacro:arg name="gpio_config" default=""/>
+  <xacro:kuka_iontec_ros2_control name="$(arg prefix)kr50_r2100" driver_version="$(arg driver_version)" client_ip="$(arg client_ip)" mxa_client_port="$(arg mxa_client_port)" controller_ip="$(arg controller_ip)" client_port="$(arg client_port)" prefix="$(arg prefix)" mode="$(arg mode)" use_gpio="$(arg use_gpio)" gpio_config="$(arg gpio_config)" roundtrip_time="$(arg roundtrip_time)" verify_robot_model="$(arg verify_robot_model)">
+    <ext_axes_ros2_control_joints/>
+  </xacro:kuka_iontec_ros2_control>
+  <!-- world link -->
+  <link name="world"/>
+  <!-- robot links, joints -->
+  <xacro:kuka_kr50_r2100_robot prefix="$(arg prefix)" package_name="kuka_iontec_support"/>
+  <!-- default world - base_link joint -->
+  <joint name="$(arg prefix)world-base_link" type="fixed">
+    <parent link="world"/>
+    <child link="$(arg prefix)base_link"/>
     <origin xyz="$(arg x) $(arg y) $(arg z)" rpy="$(arg roll) $(arg pitch) $(arg yaw)"/>
-  </xacro:kuka_kr50_r2100_robot>
+  </joint>
 </robot>

File: kuka_iontec_support/urdf/kr50_r2100_macro.xacro (robot description, xacro)
@@ -1,7 +1,6 @@
 <?xml version="1.0"?>
 <robot xmlns:xacro="http://wiki.ros.org/xacro">
-  <xacro:macro name="kuka_kr50_r2100_robot" params="prefix package_name link_6_es_angle:=0.0 *origin">
+  <xacro:macro name="kuka_kr50_r2100_robot" params="prefix package_name link_6_es_angle:=0.0">
     <!-- links - main serial chain -->
-    <link name="world"/>
     <link name="${prefix}base_link">
       <collision>
@@ -155,9 +154,4 @@
       </visual>
     </link>
-    <joint name="${prefix}world-base_link" type="fixed">
-      <parent link="world"/>
-      <child link="${prefix}base_link"/>
-      <xacro:insert_block name="origin"/>
-    </joint>
     <joint name="${prefix}joint_1" type="revolute">
       <axis xyz="0.0 0.0 1.0"/>
