Commit message: Allow new robot-rail mounting orientations

File: kuka_kl_support/urdf/kl100_2_macro.xacro (robot description, xacro)
@@ -28,5 +28,5 @@
     </link>
   </xacro:macro>
-  <xacro:macro name="kl100_2_joints" params="robot_base_link *origin">
+  <xacro:macro name="kl100_2_joints" params="robot_base_link yaw_kl_robot:=0.0 *origin">
     <!-- joints -->
     <joint name="world-rail_base" type="fixed">
@@ -45,5 +45,5 @@
       <parent link="rail_moving_link"/>
       <child link="${robot_base_link}"/>
-      <origin rpy="0.0 0.0 0.0" xyz="0.0 0.0 0.356"/>
+      <origin rpy="0.0 0.0 ${yaw_kl_robot}" xyz="0.0 0.0 0.356"/>
     </joint>
   </xacro:macro>
