Commit message: Update kl limits

File: kuka_kl_support/urdf/kl4000_macro.xacro (robot description, xacro)
@@ -58,5 +58,5 @@
       <origin rpy="0.0 0.0 0.0" xyz="0.0 0.0 0.0"/>
       <axis xyz="1 0 0"/>
-      <limit lower="-1.0" upper="1.0" effort="702.0" velocity="2.5"/>
+      <limit lower="-2.0" upper="0.0" effort="702.0" velocity="2.5"/>
     </joint>
     <joint name="rail-adapter_plate" type="fixed">

Commit message: Update kl4000

File: kuka_kl_support/urdf/kl4000_macro.xacro (robot description, xacro)
@@ -9,5 +9,5 @@
       <visual>
         <geometry>
-          <mesh filename="package://kuka_kl_support/meshes/kl4000/visual/KL4000_lange_Kette_BK309_fixed.stl" scale="0.001 0.001 0.001"/>
+          <mesh filename="package://kuka_kl_support/meshes/kl4000/visual/rail_base_link.dae"/>
         </geometry>
         <material name="dark_grey"/>
@@ -15,5 +15,5 @@
       <collision>
         <geometry>
-          <mesh filename="package://kuka_kl_support/meshes/kl4000/collision/KL4000_lange_Kette_BK309_fixed.stl" scale="0.001 0.001 0.001"/>
+          <mesh filename="package://kuka_kl_support/meshes/kl4000/collision/rail_base_link.stl"/>
         </geometry>
       </collision>
@@ -22,5 +22,5 @@
       <visual>
         <geometry>
-          <mesh filename="package://kuka_kl_support/meshes/kl4000/visual/KL4000_lange_Kette_BK309_movinglink.stl" scale="0.001 0.001 0.001"/>
+          <mesh filename="package://kuka_kl_support/meshes/kl4000/visual/rail_moving_link.dae"/>
         </geometry>
         <material name="dark_grey"/>
@@ -28,5 +28,5 @@
       <collision>
         <geometry>
-          <mesh filename="package://kuka_kl_support/meshes/kl4000/collision/KL4000_lange_Kette_BK309_movinglink.stl" scale="0.001 0.001 0.001"/>
+          <mesh filename="package://kuka_kl_support/meshes/kl4000/collision/rail_moving_link.stl"/>
         </geometry>
       </collision>
@@ -35,11 +35,10 @@
       <visual>
         <geometry>
-          <mesh filename="package://kuka_kl_support/meshes/kl4000/visual/Zwischenplatte_Quantec.stl" scale="0.001 0.001 0.001"/>
+          <mesh filename="package://kuka_kl_support/meshes/kl4000/visual/AdapterPlate_Iontec.dae"/>
         </geometry>
-        <material name="dark_grey"/>
       </visual>
       <collision>
         <geometry>
-          <mesh filename="package://kuka_kl_support/meshes/kl4000/collision/Zwischenplatte_Quantec.stl" scale="0.001 0.001 0.001"/>
+          <mesh filename="package://kuka_kl_support/meshes/kl4000/collision/AdapterPlate_Iontec.stl"/>
         </geometry>
       </collision>
@@ -58,5 +57,5 @@
       <origin rpy="0.0 0.0 0.0" xyz="0.0 0.0 0.0"/>
       <axis xyz="1 0 0"/>
-      <limit lower="-2.0" upper="0.0" effort="702.0" velocity="2.5"/>
+      <limit lower="-2.170" upper="0.175" effort="702.0" velocity="2.5"/>
     </joint>
     <joint name="rail-adapter_plate" type="fixed">
